Commit message: Add dummy collision to avoid moveit warnings

File: velodyne_description/urdf/HDL-32E.urdf.xacro (robot description, xacro)
@@ -45,4 +45,9 @@
         </geometry>
       </visual>
+      <collision>
+        <geometry>
+          <sphere radius="0"/>
+        </geometry>
+      </collision>
     </link>
     <!-- Gazebo requires the velodyne_gazebo_plugins package -->

File: velodyne_description/urdf/VLP-16.urdf.xacro (robot description, xacro)
@@ -50,4 +50,9 @@
         </geometry>
       </visual>
+      <collision>
+        <geometry>
+          <sphere radius="0"/>
+        </geometry>
+      </collision>
     </link>
     <!-- Gazebo requires the velodyne_gazebo_plugins package -->
